File: mbi5029_led_matrix.kicad_pcb (KiCad board)
At the start: 4 copper layers, 277 parts, among them Q1 pCh SO23, Q10 pCh SO23, Q11 pCh SO23, Q12 pCh SO23, Q13 pCh SO23, Q14 pCh SO23, Q15 pCh SO23, Q16 pCh SO23, Q2 pCh SO23, Q3 pCh SO23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

Commit message: work
Parts:
- removed N1: OHWLOGO, Symbols:OSHW-Symbol_6.7x6mm_SilkScreen
- removed N2: V20171120, SquantorLabels:Label_version
- moved D241 184.4 mm to (184.2, 63.0), turned to 45 degrees
- moved U2 183.8 mm to (210.2, 86.3)
- moved U3 183.8 mm to (210.2, 97.8)
- moved D242 181.2 mm to (184.2, 66.8), turned to 45 degrees
- moved D225 180.9 mm to (180.3, 63.0), turned to 45 degrees
- moved D243 178.1 mm to (184.2, 70.6), turned to 45 degrees
- moved D226 177.7 mm to (180.3, 66.8), turned to 45 degrees
- moved D209 177.4 mm to (176.5, 63.0), turned to 45 degrees
- moved D244 175.0 mm to (184.2, 74.4), turned to 45 degrees
- moved D227 174.7 mm to (180.3, 70.6), turned to 45 degrees
- moved D210 174.3 mm to (176.5, 66.8), turned to 45 degrees
- moved D193 174.0 mm to (172.7, 63.0), turned to 45 degrees
- moved D245 172.1 mm to (184.2, 78.2), turned to 45 degrees
- moved D228 171.7 mm to (180.3, 74.4), turned to 45 degrees
- moved D211 171.4 mm to (176.5, 70.6), turned to 45 degrees
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Connections:
- U1 pad 1: unconnected-(U1-Pad1) -> GND
- U1 pad 2: unconnected-(U1-Pad2) -> (no net)
- U1 pad 21: unconnected-(U1-Pad21) -> (no net)
- U1 pad 22: unconnected-(U1-Pad22) -> (no net)
- U1 pad 23: unconnected-(U1-Pad23) -> (no net)
- U1 pad 24: unconnected-(U1-Pad24) -> +5V
- U1 pad 3: unconnected-(U1-Pad3) -> (no net)
- U1 pad 4: unconnected-(U1-Pad4) -> (no net)
- U2 pad 1: unconnected-(U2-Pad1) -> (no net)
- U2 pad 10: unconnected-(U2-Pad10) -> /G_13
- U2 pad 11: unconnected-(U2-Pad11) -> /G_12
- U2 pad 12: unconnected-(U2-Pad12) -> /G_11
- U2 pad 13: unconnected-(U2-Pad13) -> /G_10
- U2 pad 14: unconnected-(U2-Pad14) -> /G_9
- U2 pad 15: unconnected-(U2-Pad15) -> /G_8
- U2 pad 16: unconnected-(U2-Pad16) -> +5V
- U2 pad 2: unconnected-(U2-Pad2) -> (no net)
- U2 pad 3: unconnected-(U2-Pad3) -> (no net)
- U2 pad 4: unconnected-(U2-Pad4) -> (no net)
- U2 pad 5: unconnected-(U2-Pad5) -> (no net)
- U2 pad 6: unconnected-(U2-Pad6) -> (no net)
- U2 pad 7: unconnected-(U2-Pad7) -> (no net)
- U2 pad 8: unconnected-(U2-Pad8) -> GND
- U2 pad 9: unconnected-(U2-Pad9) -> /G_14
- U3 pad 1: unconnected-(U3-Pad1) -> (no net)
- U3 pad 10: unconnected-(U3-Pad10) -> /G_5
- U3 pad 11: unconnected-(U3-Pad11) -> /G_4
- U3 pad 12: unconnected-(U3-Pad12) -> /G_3
- U3 pad 13: unconnected-(U3-Pad13) -> /G_2
- U3 pad 14: unconnected-(U3-Pad14) -> /G_1
- U3 pad 15: unconnected-(U3-Pad15) -> /G_0
- U3 pad 16: unconnected-(U3-Pad16) -> +5V
- U3 pad 2: unconnected-(U3-Pad2) -> (no net)
- U3 pad 3: unconnected-(U3-Pad3) -> (no net)
- U3 pad 4: unconnected-(U3-Pad4) -> (no net)
- U3 pad 5: unconnected-(U3-Pad5) -> (no net)
- U3 pad 6: unconnected-(U3-Pad6) -> (no net)
- U3 pad 7: unconnected-(U3-Pad7) -> /G_7
- U3 pad 8: unconnected-(U3-Pad8) -> GND
- U3 pad 9: unconnected-(U3-Pad9) -> /G_6
Routing:
- net /LED Matrix 16x16/LED_K0: track 0.00 -> 101.5 mm
- net /LED Matrix 16x16/LED_K1: track 0.00 -> 96.5 mm
- net /LED Matrix 16x16/LED_K8: track 0.00 -> 93.2 mm
- net /LED Matrix 16x16/LED_K2: track 0.00 -> 90.4 mm
- net /LED Matrix 16x16/LED_K9: track 0.00 -> 88.2 mm
- net /LED Matrix 16x16/LED_K11: track 0.00 -> 86.1 mm
- net /LED Matrix 16x16/LED_K10: track 0.00 -> 85.9 mm
- net /LED Matrix 16x16/LED_K3: track 0.00 -> 85.9 mm
- net /LED_A9: track 0.00 -> 83.6 mm, vias 0 -> 16
- net /LED_A8: track 0.00 -> 83.6 mm, vias 0 -> 16
- net /LED_A7: track 0.00 -> 83.6 mm, vias 0 -> 16
- net /LED_A6: track 0.00 -> 83.6 mm, vias 0 -> 16
- net /LED_A5: track 0.00 -> 83.6 mm, vias 0 -> 16
- net /LED_A4: track 0.00 -> 83.6 mm, vias 0 -> 16
- net /LED_A3: track 0.00 -> 83.6 mm, vias 0 -> 16
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
Commit message: more work!
Parts:
- added C1: 100n, Capacitor_SMD:C_0603_1608Metric, F.Cu at (204.7, 74.7)
- added C2: 100n, Capacitor_SMD:C_0603_1608Metric, F.Cu at (197.6, 108.2)
- added C3: 100n, Capacitor_SMD:C_0603_1608Metric, F.Cu at (197.6, 73.7)
- added J1: Conn_02x08_Odd_Even, Connector_PinHeader_2.54mm:PinHeader_2x08_P2.54mm_Vertical, F.Cu at (209.8, 102.1)
- moved D1 80.8 mm to (184.2, 120.2)
- moved D16 80.8 mm to (184.2, 63.0)
- moved D241 80.8 mm to (127.0, 120.2)
- moved D256 80.8 mm to (127.0, 63.0)
- moved D15 75.6 mm to (184.2, 66.8)
- moved D17 75.6 mm to (180.3, 120.2)
- moved D2 75.6 mm to (184.2, 116.3)
- moved D225 75.6 mm to (130.8, 120.2)
- moved D240 75.6 mm to (130.8, 63.0)
- moved D242 75.6 mm to (127.0, 116.3)
- moved D255 75.6 mm to (127.0, 66.8)
- moved D32 75.6 mm to (180.3, 63.0)
- moved D14 70.9 mm to (184.2, 70.6)
- moved D209 70.9 mm to (134.6, 120.2)
- moved D224 70.9 mm to (134.6, 63.0)
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Connections:
- Q14 pad 1: /G_12 -> /G_13
- Q15 pad 1: /G_13 -> /G_14
- Q16 pad 1: /G_14 -> /G_15
- U2 pad 1: (no net) -> /A0
- U2 pad 2: (no net) -> /A1
- U2 pad 3: (no net) -> /A2
- U2 pad 7: (no net) -> /G_15
- U3 pad 1: (no net) -> /A0
- U3 pad 2: (no net) -> /A1
- U3 pad 3: (no net) -> /A2
Routing:
- net /LED Matrix 16x16/LED_K15: track 61.0 -> 193.1 mm, vias 0 -> 2
- net /LED Matrix 16x16/LED_K14: track 61.0 -> 191.7 mm, vias 0 -> 2
- net /LED Matrix 16x16/LED_K13: track 61.0 -> 186.9 mm, vias 0 -> 2
- net /LED Matrix 16x16/LED_K12: track 75.6 -> 181.9 mm, vias 0 -> 2
- net /LED Matrix 16x16/LED_K11: track 86.1 -> 180.7 mm, vias 0 -> 2
- net /LED Matrix 16x16/LED_K10: track 85.9 -> 174.6 mm, vias 0 -> 2
- net /LED Matrix 16x16/LED_K7: track 70.7 -> 159.2 mm, vias 0 -> 2
- net /LED_A8: track 83.6 -> 171.8 mm, vias 16 -> 33
- net /LED_A12: track 83.6 -> 171.8 mm, vias 16 -> 33
- net /LED_A9: track 83.6 -> 171.8 mm, vias 16 -> 33
- net /LED_A7: track 83.6 -> 171.8 mm, vias 16 -> 33
- net /LED_A5: track 83.6 -> 171.8 mm, vias 16 -> 33
- net /LED_A4: track 83.6 -> 171.8 mm, vias 16 -> 33
- net /LED_A3: track 83.6 -> 171.8 mm, vias 16 -> 33
- net /LED_A2: track 83.6 -> 171.8 mm, vias 16 -> 33
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- added copper zone on In1.Cu, net +5V
- added copper zone on In2.Cu, net GND

Commit message: more work
Parts:
- added C4: 100n, Capacitor_SMD:C_0603_1608Metric, F.Cu at (202.9, 109.7)
- added C5: 100n, Capacitor_SMD:C_0603_1608Metric, F.Cu at (214.1, 109.7)
- added R1: 1k, Resistor_SMD:R_0603_1608Metric, F.Cu at (207.3, 74.7)
- added R2: 1k, Resistor_SMD:R_0603_1608Metric, F.Cu at (211.8, 92.5)
- added R3: 1k, Resistor_SMD:R_0603_1608Metric, F.Cu at (211.8, 90.7)
- added R4: 1k, Resistor_SMD:R_0603_1608Metric, F.Cu at (211.8, 88.9)
- added R5: 1k, Resistor_SMD:R_0603_1608Metric, F.Cu at (211.8, 87.1)
- added R6: 1k, Resistor_SMD:R_0603_1608Metric, F.Cu at (211.8, 85.3)
- added U4: 74HCT14, Package_SO:SOIC-14_3.9x8.7mm_P1.27mm, F.Cu at (211.6, 116.1)
- added U5: 74HCT595, Package_SO:SOIC-16_3.9x9.9mm_P1.27mm, F.Cu at (200.0, 116.7)
- J1: value Conn_02x08_Odd_Even -> Conn_02x04_Odd_Even; footprint Connector_PinHeader_2.54mm:PinHeader_2x08_P2.54mm_Vertical -> Connector_PinHeader_2.54mm:PinHeader_2x04_P2.54mm_Vertical
- U1: value MBI5029 -> mbi5029gd; footprint Package_SO:SO-24_5.3x15mm_P1.27mm -> Package_SO:SOIC-24W_7.5x15.4mm_P1.27mm
- U2, U3: value 74HC237 -> 74HCT137
- moved J1 5.59 mm to (209.8, 96.5)
- moved U1 1.02 mm to (202.2, 84.3)
Connections:
- J1 pad 1: (no net) -> GND
- J1 pad 2: (no net) -> /~{COPI_LV}
- J1 pad 3: (no net) -> /~{CIPO}
- J1 pad 4: (no net) -> /~{LE_LV}
- J1 pad 5: (no net) -> /K_OE_LV
- J1 pad 6: (no net) -> /AN_OE_LV
- J1 pad 7: (no net) -> /~{SCLK_LV}
- J1 pad 8: (no net) -> GND
- U1 pad 2: (no net) -> /COPI
- U1 pad 21: (no net) -> /~{K_OE}
- U1 pad 22: (no net) -> /SD_MID
- U1 pad 23: (no net) -> Net-(U1-Pad23)
- U1 pad 3: (no net) -> /SCLK
- U1 pad 4: (no net) -> /LE
- U2 pad 4: (no net) -> GND
- U2 pad 5: (no net) -> /~{AN_OE}
- U2 pad 6: (no net) -> /E_AN2
- U3 pad 4: (no net) -> GND
- U3 pad 5: (no net) -> /~{AN_OE}
- U3 pad 6: (no net) -> /E_AN1
Routing:
- net /~{AN_OE}: track 0.00 -> 80.1 mm, vias 0 -> 6
- net /E_AN2: track 0.00 -> 61.2 mm
- net /LE: track 0.00 -> 56.8 mm, vias 0 -> 5
- net /COPI: track 0.00 -> 53.6 mm, vias 0 -> 2
- net /SCLK: track 0.00 -> 53.0 mm, vias 0 -> 2
- net /~{K_OE}: track 0.00 -> 52.0 mm, vias 0 -> 2
- net /SD_MID: track 0.00 -> 44.7 mm, vias 0 -> 2
- net /~{SCLK_LV}: track 0.00 -> 41.1 mm, vias 0 -> 1
- net /K_OE_LV: track 0.00 -> 38.1 mm, vias 0 -> 1
- net /AN_OE_LV: track 0.00 -> 35.5 mm, vias 0 -> 1
- net /~{LE_LV}: track 0.00 -> 31.1 mm
- net /CIPO: track 0.00 -> 26.2 mm, vias 0 -> 2
- net /E_AN1: track 0.00 -> 23.7 mm
- net /~{CIPO}: track 0.00 -> 23.6 mm, vias 0 -> 1
- net /~{COPI_LV}: track 0.00 -> 23.4 mm
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