File: mbi5029_led_matrix.kicad_sch (KiCad schematic)
At the start: 19 parts, among them Q1 pCh SO23, Q10 pCh SO23, Q11 pCh SO23, Q12 pCh SO23, Q13 pCh SO23, Q14 pCh SO23, Q15 pCh SO23, Q16 pCh SO23, Q2 pCh SO23, Q3 pCh SO23, Q4 pCh SO23, Q5 pCh SO23, Q6 pCh SO23, Q7 pCh SO23, Q8 pCh SO23, Q9 pCh SO23, U1 MBI5029, U2 74HC237, U3 74HC237

Commit message: work
Parts:
- added J?: Conn_02x08_Odd_Even, symbol Connector_Generic:Conn_02x08_Odd_Even
Connections:
- net +5V: now also U1.24 (VDD), U2.16 (VCC), U3.16 (VCC)
- net G_0: now also U3.15 (Y0)
- net G_1: now also U3.14 (Y1)
- net G_10: now also U2.13 (Y2)
- net G_11: now also U2.12 (Y3)
- net G_12: now also U2.11 (Y4)
- net G_13: now also U2.10 (Y5)
- net G_14: now also U2.9 (Y6)
- net G_2: now also U3.13 (Y2)
- net G_3: now also U3.12 (Y3)
- net G_4: now also U3.11 (Y4)
- net G_5: now also U3.10 (Y5)
- net G_6: now also U3.9 (Y6)
- net G_7: now also U3.7 (Y7)
- net G_8: now also U2.15 (Y0)
- net G_9: now also U2.14 (Y1)
- net GND: now reaches U3.8 (GND)
- net GND: now also U1.1 (GND), U2.8 (GND)
- net G_15: now reaches U2.7 (Y7)
Other:
- moved on the sheet: U1, U2, U3

Commit message: more work!
Parts:
- added C1, C2, C3: 100n, Capacitor_SMD:C_0603_1608Metric, symbol Device:C
- added U4: 74HC14, symbol 74xx:74HC14
- J1: renamed from J?; footprint (none) -> Connector_PinHeader_2.54mm:PinHeader_2x08_P2.54mm_Vertical
Connections:
- net +5V: now also C1.2, C2.2, C3.2
- net GND: now also C1.1, C2.1, C3.1
- net G_12: no longer Q14.1 (G)
- net G_13: now also Q14.1 (G); no longer Q15.1 (G)
- net G_14: now also Q15.1 (G); no longer Q16.1 (G)
- net G_15: now also Q16.1 (G)
- net A0: now reaches U3.1 (A0)
- net A0: now also U2.1 (A0)
- net A1: now reaches U3.2 (A1)
- net A1: now also U2.2 (A1)
- net A2: now reaches U3.3 (A2)
- net A2: now also U2.3 (A2)

Commit message: more work
Parts:
- removed J1: Conn_02x08_Odd_Even, Connector_PinHeader_2.54mm:PinHeader_2x08_P2.54mm_Vertical, symbol Connector_Generic:Conn_02x08_Odd_Even
- removed U1: MBI5029, Package_SO:SO-24_5.3x15mm_P1.27mm, symbol Driver_LED:STP16CP05
- removed U2: 74HC237, Package_SO:SOIC-16_3.9x9.9mm_P1.27mm, symbol 74xx:74HC237
- added C4, C5: 100n, Capacitor_SMD:C_0603_1608Metric, symbol Device:C
- added J1: Conn_02x04_Odd_Even, Connector_PinHeader_2.54mm:PinHeader_2x04_P2.54mm_Vertical, symbol Connector_Generic:Conn_02x04_Odd_Even
- added R1, R2, R3, R4, R5, R6: 1k, Resistor_SMD:R_0603_1608Metric, symbol Device:R
- added U1: mbi5029gd, Package_SO:SOIC-24W_7.5x15.4mm_P1.27mm, symbol mbi5029_led_matrix:mbi5029gd
- added U2: 74HCT137, Package_SO:SOIC-16_3.9x9.9mm_P1.27mm, symbol 74xx:74HCT137
- added U5: 74HCT595, Package_SO:SOIC-16_3.9x9.9mm_P1.27mm, symbol 74xx:74HCT595
- U3: value 74HC237 -> 74HCT137; symbol 74xx:74HC237 -> 74xx:74HCT137
- U4: value 74HC14 -> 74HCT14; footprint (none) -> Package_SO:SOIC-14_3.9x8.7mm_P1.27mm
Connections:
- net +5V: now also U4.14 (VCC), C4.2, C5.2, R1.1, U1.24 (VDD), U2.16 (VCC), U5.10 (~{SRCLR}), U5.16 (VCC)
- net A0: now also U2.1 (A0), U5.15 (QA)
- net A1: now also U2.2 (A1), U5.1 (QB)
- net A2: now also U2.3 (A2), U5.2 (QC)
- net GND: now also U3.4 (~{LE}), U4.7 (GND), C4.1, C5.1, J1.1 (Pin_1), J1.8 (Pin_8), R2.2, R3.2, R4.2, R5.2, R6.2, U1.1 (GND), U2.4 (~{LE}), U2.8 (GND), U5.13 (~{OE}), U5.8 (GND)
- net G_10: now also U2.13 (~{Y2})
- net G_11: now also U2.12 (~{Y3})
- net G_12: now also U2.11 (~{Y4})
- net G_13: now also U2.10 (~{Y5})
- net G_14: now also U2.9 (~{Y6})
- net G_15: now also U2.7 (~{Y7})
- net G_8: now also U2.15 (~{Y0})
- net G_9: now also U2.14 (~{Y1})
- net LED_K0: now also U1.5 (~{OUT0})
- net LED_K1: now also U1.6 (~{OUT1})
- net LED_K10: now also U1.15 (~{OUT10})
- net LED_K11: now also U1.16 (~{OUT11})
- net LED_K12: now also U1.17 (~{OUT12})
- net LED_K13: now also U1.18 (~{OUT13})
- net LED_K14: now also U1.19 (~{OUT14})
- net LED_K15: now also U1.20 (~{OUT15})
- net LED_K2: now also U1.7 (~{OUT2})
- net LED_K3: now also U1.8 (~{OUT3})
- net LED_K4: now also U1.9 (~{OUT4})
- net LED_K5: now also U1.10 (~{OUT5})
- net LED_K6: now also U1.11 (~{OUT6})
- net LED_K7: now also U1.12 (~{OUT7})
- net LED_K8: now also U1.13 (~{OUT8})
- net LED_K9: now also U1.14 (~{OUT9})
- net ~{COPI_LV}: now reaches U4.1
- net ~{COPI_LV}: now also J1.2 (Pin_2), R2.1
- net COPI: now reaches U4.2
- net COPI: now also U1.2 (SDI)
- net ~{AN_OE}: now reaches U4.10
- net ~{AN_OE}: now also U3.5 (~{E1}), U2.5 (~{E1})
- net AN_OE_LV: now reaches U4.11
- net AN_OE_LV: now also J1.6 (Pin_6), R5.1
- net ~{SCLK_LV}: now reaches U4.5
- net ~{SCLK_LV}: now also J1.7 (Pin_7), R6.1
- net SCLK: now reaches U4.6
- net SCLK: now also U1.3 (CLK), U5.11 (SRCLK)
- net E_AN1: now reaches U3.6 (E2)
- net E_AN1: now also U5.3 (QD)
- net ~{CIPO}: now reaches U4.12
- net ~{CIPO}: now also J1.3 (Pin_3)
- net CIPO: now reaches U4.13
- net CIPO: now also U5.9 (QH')
- net ~{LE_LV}: now reaches U4.3
- net ~{LE_LV}: now also J1.4 (Pin_4), R3.1
- net LE: now reaches U4.4
- net LE: now also U1.4 (LE/MOD/CA), U5.12 (RCLK)
- net ~{K_OE}: now reaches U4.8
- net ~{K_OE}: now also U1.21 (~{OE}/SW/~{ED})
- net K_OE_LV: now reaches U4.9
- net K_OE_LV: now also J1.5 (Pin_5), R4.1
- new net: R1.2, U1.23 (R-EXT)
- new net E_AN2: U2.6 (E2), U5.4 (QE)
- new net SD_MID: U1.22 (SDO), U5.14 (SER)
Other:
- moved on the sheet: C1
